Commit message: FIX: frame orientation

File: data/urdf/air_humanoid.urdf (robot description, URDF)
Before this commit: robot air-humanoid, 27 links, 26 joints
Links:
- link arm_left_shoulder_pitch: mass 0.55801102950394643187 -> 0.5580110295039465429
- link arm_right_shoulder_pitch: mass 0.55801102950394643187 -> 0.5580110295039465429
- link chest: mass 1.8257137134967265091 -> 1.8257137134967282854
- link head: mass 0.38902069422263646503 -> 0.38902069422263652054
- link leg_left_feet: mass 0.15372739596032980458 -> 0.15372739596032983234
- link leg_left_hip_pitch: mass 0.55801102950394643187 -> 0.5580110295039465429
- link leg_left_hip_roll: mass 0.55801102950394643187 -> 0.5580110295039465429
- link leg_left_hip_yaw: mass 0.23766371464345462106 -> 0.23766371464345470432
- link leg_left_knee: mass 0.55801102950394643187 -> 0.5580110295039465429
- link leg_right_hip_pitch: mass 0.55801102950394643187 -> 0.5580110295039465429
- link leg_right_hip_roll: mass 0.55801102950394643187 -> 0.5580110295039465429
- link leg_right_hip_yaw: mass 0.23766122387422328188 -> 0.23766122387422336515
- link leg_right_knee: mass 0.55801102950394643187 -> 0.5580110295039465429
- link pelvis: mass 1.3501169634884675474 -> 1.3501169634884679915
- link right_hand: mass 0.068213107958726204583 -> 0.068213107958726190705
Joints:
- joint arm_left_elbow_pitch_joint: origin xyz=-2.7755575615628913511e-17 0 -0.14999999999999996669 rpy=-1.4093274315810776596e-15 1.5707963267948927832 0 -> xyz=4.7184478546569152968e-16 0 -0.15000000000000004996 rpy=9.58456417818011379e-16 1.5707963267948876762 0
- joint arm_left_shoulder_pitch_joint: origin xyz=-0.066000000000000016986 -0.018000000000000002109 0.21749999999999997113 rpy=2.1545200642171113924e-32 1.570796326794896336 0 -> xyz=-0.066000000000000003109 -0.018000000000000005579 0.21749999999999997113 rpy=-1.5729177094632718635e-31 1.570796326794896336 0
- joint arm_left_shoulder_roll_joint: origin xyz=0 0 0 rpy=-1.570796326794896558 -1.0471975511965940786 2.2204460492503170252e-16 -> xyz=0 3.4694469519536141888e-18 0 rpy=-1.5707963267948952257 -1.0471975511965974093 5.2973253724013804362e-16
- joint arm_left_shoulder_yaw_joint: origin xyz=0 0 -3.4694469519536141888e-18 rpy=1.570796326794896336 -9.2721311233901574007e-15 -1.7010002593405239514e-17 -> xyz=-2.7755575615628913511e-17 2.7755575615628913511e-17 0 rpy=1.570796326794896336 7.4222288895831854852e-18 -1.9051709141231696514e-15
- joint arm_left_wrist_yaw_joint: origin xyz=0.14999999999999996669 -3.4694469519536141888e-18 -2.7755575615628913511e-17 rpy=3.9315131168840358984e-30 -1.5707963267948938935 0 -> xyz=0.14999999999999996669 0 -2.7755575615628913511e-17 rpy=-9.8482095003098587547e-31 -1.5707963267948870101 0
- joint arm_right_elbow_pitch_joint: origin xyz=5.5511151231257827021e-17 0 -0.1500000000000000222 rpy=-1.6024377162891802108e-30 1.5707963267948958919 0 -> xyz=-8.3266726846886740532e-17 0 -0.14999999999999999445 rpy=-2.1372674594763257107e-18 1.5707963267948941155 0
- joint arm_right_shoulder_pitch_joint: origin xyz=0.065999999999999989231 -0.018000000000000002109 0.21750000000000002665 rpy=6.1443752211428073199e-32 1.570796326794896336 0 -> xyz=0.066000000000000016986 -0.017999999999999988232 0.21750000000000002665 rpy=-6.9714611098467086935e-32 1.570796326794896336 0
- joint arm_right_shoulder_roll_joint: origin xyz=1.1102230246251565404e-16 0 1.1102230246251565404e-16 rpy=1.5707963267948961139 -1.0471975511965978534 -3.141592653589793116 -> xyz=4.4408920985006261617e-16 0 1.9428902930940239457e-16 rpy=1.5707963267948958919 -1.0471975511965982975 -3.1415926535897908956
- joint arm_right_shoulder_yaw_joint: origin xyz=-2.2204460492503130808e-16 -1.3877787807814456755e-16 0 rpy=1.570796326794896336 2.0065992624732387539e-29 -6.4961943429070360185e-16 -> xyz=0 2.7755575615628913511e-17 0 rpy=1.570796326794896336 -5.923750470296498874e-15 -1.1874347964521361147e-15
- joint arm_right_wrist_yaw_joint: origin xyz=0.15000000000000712763 -2.3939183968479937903e-16 6.0507154842071031453e-15 rpy=-1.4011522297361927018e-27 -1.570796326794896558 0 -> xyz=0.14999999999999769074 3.4694469519536141888e-18 -1.3877787807814456755e-16 rpy=-1.3808453847752483308e-31 -1.570796326794891673 0
- joint leg_left_ankle_pitch_joint: origin xyz=0 -3.4694469519536141888e-18 3.3306690738754696213e-16 rpy=-1.0179494176688816214e-16 1.5707963267948925612 0 -> xyz=-6.9388939039072283776e-18 0 1.1102230246251565404e-16 rpy=-3.4943327596190197446e-17 1.5707963267948845676 0
- joint leg_left_ankle_roll_joint: origin xyz=-1.1102230246251565404e-16 0 1.3877787807814456755e-17 rpy=-1.570796326794896336 -1.570796326794896336 0 -> xyz=0 0 0 rpy=-1.570796326794896336 -1.5707963267948832353 0
- joint leg_left_ankle_yaw_joint: origin xyz=0.29250000000000014877 -0.022499999999999995698 -6.2450045135165055399e-17 rpy=1.6294908073472161295e-29 -1.5707963267948927832 0 -> xyz=0.29250000000000009326 -0.022499999999999999167 -6.2450045135165055399e-17 rpy=-1.5796939627050750193e-28 -1.5707963267948790165 0
- joint leg_left_hip_pitch_joint: origin xyz=-0.053999999999999999389 1.6177811532852781166e-32 2.3980817331903381002e-17 rpy=1.7137261189858739291e-24 1.5707963267948947816 0 -> xyz=-9.254121991410917654e-26 0.053999999999999999389 2.3980817331903381002e-17 rpy=1.570796326794896558 1.5707963267948947816 0
- joint leg_left_hip_roll_joint: origin xyz=-8.9363149419567743582e-32 -4.1382979265456836971e-16 0 rpy=-1.570796326794896336 -1.5707963267948954478 0 -> xyz=-1.6948183510607675507e-32 2.5038415798651811879e-18 0 rpy=-1.570796326794896336 -1.570796326794896336 0
- joint leg_left_hip_yaw_joint: origin xyz=0 0 0 rpy=1.570796326794896336 -2.1788126875405682641e-15 4.3796597585432577988e-15 -> xyz=0 -2.9774503199148973655e-31 3.8518598887744717061e-34 rpy=1.570796326794896336 1.2656542480726820848e-14 -6.1232339957379111168e-17
- joint leg_left_knee_pitch_joint: origin xyz=0 4.1382979265456600312e-16 -0.25500000000000000444 rpy=6.0273563179670801322e-31 1.5707963267948923392 0 -> xyz=0 -9.8607613152626475676e-32 -0.25500000000000000444 rpy=6.8009041934528729891e-31 1.570796326794896558 0
- joint leg_right_ankle_pitch_joint: origin xyz=-8.3266726846886740532e-17 -3.4694469519536141888e-18 1.1102230246251565404e-16 rpy=-3.7358416039018505946e-31 1.570796326794896558 0 -> xyz=0 -6.9388939039072283776e-18 1.1102230246251565404e-16 rpy=-9.7085368725430385662e-31 1.570796326794896336 0
- joint leg_right_ankle_roll_joint: origin xyz=0 0 6.9388939039072283776e-18 rpy=-1.5707963267948978903 -1.570796326794896558 0 -> xyz=1.1102230246251565404e-16 1.0408340855860842566e-17 -6.9388939039072283776e-18 rpy=-1.570796326794896336 -1.570796326794896336 0
- joint leg_right_ankle_yaw_joint: origin xyz=0.29250000000000014877 -0.022499999999999995698 9.0205620750793968909e-17 rpy=1.2284259059637670751e-29 -1.570796326794896558 0 -> xyz=0.29249999999999992673 -0.022499999999999995698 -6.9388939039072283776e-17 rpy=-7.0041171194910210604e-16 -1.5707963267948945596 0
- joint leg_right_hip_pitch_joint: origin xyz=0.053999999999999999389 -1.6948183510607675507e-32 -2.0816681711721685133e-17 rpy=6.902532920683827023e-31 1.570796326794896336 0 -> xyz=-1.2575511642735519166e-30 -0.053999999999999999389 -2.3980817331903381002e-17 rpy=1.570796326794896558 1.5707963267948947816 0
- joint leg_right_hip_roll_joint: origin xyz=-1.5407439555097886824e-33 5.4738221262688166833e-48 6.9388939039072283776e-18 rpy=-1.570796326794896558 -1.570796326794896336 0 -> xyz=7.4767711785223679523e-18 -2.5533811274267894e-19 0 rpy=-1.570796326794896336 -1.570796326794896336 0
- joint leg_right_hip_yaw_joint: origin xyz=-1.3877787807814456755e-17 6.5481618109166019004e-33 -2.3111159332646830237e-33 rpy=1.570796326794896336 -1.7655075777304626956e-30 -1.9721522630525286377e-31 -> xyz=4.8572257327350598644e-17 -4.7184478546569152968e-16 1.6767916467813030231e-29 rpy=1.570796326794896336 3.2375344588336235604e-28 2.9582283945787877017e-31
- joint leg_right_knee_pitch_joint: origin xyz=2.0816681711721685133e-17 -1.1555579666323415118e-31 -0.25499999999999989342 rpy=1.1263763291195329189e-30 1.570796326794896336 0 -> xyz=-4.1633363423443370266e-17 1.0557947955130826946e-29 -0.25500000000000017097 rpy=4.4195767621494189214e-30 1.570796326794896336 0
- joint neck_yaw_joint: origin xyz=0 -4.7331654313260684678e-32 0.2999999999999999889 rpy=0 -0 8.7581154020301066933e-47 -> xyz=-1.9894085953542392168e-31 -7.1983557601417303597e-32 0.2999999999999999889 rpy=-1.9721522630525295135e-31 -0 -5.0132886437559447427e-30
- joint waist_yaw_joint: origin xyz=2.6645352591003755984e-17 -1.06581410364014913e-16 0.05999999999999999778 rpy=1.7763568394002486897e-15 4.4408920985006261617e-16 -3.0122599919713258989e-31 -> xyz=-1.0658141036401488835e-16 -2.664535259100376831e-17 0.05999999999999999778 rpy=1.7763568394002486897e-15 4.4408920985006261617e-16 -1.570796326794896558
