Commit message: ADD: upgrade to new onshape exporter

File: data/urdf/berkeley_humanoid_lite.urdf (robot description, URDF)
Before this commit: robot berkeley-humanoid-lite, 26 links, 25 joints
Links:
- added link imu_2, mass 0.00197704; visual mesh filename=./assets/merged/imu_2_visual.stl
- link arm_left_elbow_pitch: mass 0.416078 -> 0.443945; geometry visual mesh filename=./assets/merged/arm_left_elbow_pitch_visual.stl
- link arm_left_elbow_roll: geometry collision cylinder length=0.12 radius=0.03; visual mesh filename=./assets/merged/arm_left_elbow_roll_visual.stl
- link arm_left_hand_link: geometry visual mesh filename=./assets/merged/arm_left_hand_link_visual.stl
- link arm_left_shoulder_pitch: geometry visual mesh filename=./assets/merged/arm_left_shoulder_pitch_visual.stl
- link arm_left_shoulder_roll: mass 0.416078 -> 0.443945; geometry visual mesh filename=./assets/merged/arm_left_shoulder_roll_visual.stl
- link arm_left_shoulder_yaw: geometry collision cylinder length=0.15 radius=0.04; visual mesh filename=./assets/merged/arm_left_shoulder_yaw_visual.stl
- link arm_right_elbow_pitch: mass 0.416078 -> 0.443945; geometry visual mesh filename=./assets/merged/arm_right_elbow_pitch_visual.stl
- link arm_right_elbow_roll: geometry collision cylinder length=0.12 radius=0.03; visual mesh filename=./assets/merged/arm_right_elbow_roll_visual.stl
- link arm_right_hand_link: geometry visual mesh filename=./assets/merged/arm_right_hand_link_visual.stl
- link arm_right_shoulder_pitch: geometry visual mesh filename=./assets/merged/arm_right_shoulder_pitch_visual.stl
- link arm_right_shoulder_roll: mass 0.416078 -> 0.443945; geometry visual mesh filename=./assets/merged/arm_right_shoulder_roll_visual.stl
- link arm_right_shoulder_yaw: geometry collision cylinder length=0.15 radius=0.04; visual mesh filename=./assets/merged/arm_right_shoulder_yaw_visual.stl
- link base: mass 4.47154 -> 4.44401; geometry collision box size=0.15 0.14 0.23; visual mesh filename=./assets/merged/base_visual.stl
- link imu: mass 0.00197704 -> 1e-9; geometry 
- link leg_left_ankle_pitch: geometry visual mesh filename=./assets/merged/leg_left_ankle_pitch_visual.stl
- link leg_left_ankle_roll: mass 0.678609 -> 0.706476; geometry collision box size=0.072 0.22 0.04; visual mesh filename=./assets/merged/leg_left_ankle_roll_visual.stl
- link leg_left_hip_pitch: geometry collision cylinder length=0.13 radius=0.05; visual mesh filename=./assets/merged/leg_left_hip_pitch_visual.stl
- link leg_left_hip_roll: geometry visual mesh filename=./assets/merged/leg_left_hip_roll_visual.stl
- link leg_left_hip_yaw: geometry visual mesh filename=./assets/merged/leg_left_hip_yaw_visual.stl
- link leg_left_knee_pitch: mass 0.66094 -> 0.653864; geometry collision cylinder length=0.15 radius=0.04; visual mesh filename=./assets/merged/leg_left_knee_pitch_visual.stl
- link leg_right_ankle_pitch: geometry visual mesh filename=./assets/merged/leg_right_ankle_pitch_visual.stl
- link leg_right_ankle_roll: mass 0.678609 -> 0.706476; geometry collision box size=0.072 0.22 0.04; visual mesh filename=./assets/merged/leg_right_ankle_roll_visual.stl
- link leg_right_hip_pitch: geometry collision cylinder length=0.13 radius=0.05; visual mesh filename=./assets/merged/leg_right_hip_pitch_visual.stl
- link leg_right_hip_roll: geometry visual mesh filename=./assets/merged/leg_right_hip_roll_visual.stl
- link leg_right_hip_yaw: geometry visual mesh filename=./assets/merged/leg_right_hip_yaw_visual.stl
- link leg_right_knee_pitch: mass 0.66094 -> 0.653864; geometry collision cylinder length=0.15 radius=0.04; visual mesh filename=./assets/merged/leg_right_knee_pitch_visual.stl
Joints:
- added joint imu_frame: type fixed, parent imu_2, child imu, origin xyz=0 -6.33816e-19 0.005 rpy=0 -0 -1.90898e-31, axis 0 0 0
- joint arm_hand_r: origin xyz=0 0 0 rpy=-3.14159 0 -1.5708 -> xyz=-6.74047e-19 5.55112e-17 0 rpy=-3.14159 -9.75587e-15 -1.5708
- joint arm_left_elbow_pitch_joint: limit lower=-0 upper=1.5708 effort=20 velocity=15 -> lower=-6.16396e-13 upper=1.5708 effort=20 velocity=15; origin xyz=0.0245 0 0.043 rpy=1.5708 0 1.5708 -> xyz=0.0245 6.0295e-17 0.043 rpy=1.5708 -3.0664e-13 1.5708
- joint arm_left_elbow_roll_joint: origin xyz=0 0.123 -0.0255 rpy=-1.5708 0 0 -> xyz=-3.16213e-14 0.123 -0.0255 rpy=-1.5708 1.75811e-13 2.18496e-13
- joint arm_left_hand_l: origin xyz=0 0 0 rpy=3.14159 0 -1.5708 -> xyz=-6.31089e-30 -5.55112e-17 5.55112e-17 rpy=3.14159 2.68666e-14 -1.5708
- joint arm_left_shoulder_pitch_joint: origin xyz=0 0.133 0.164028 rpy=-1.5708 0 0 -> xyz=8.30342e-16 0.133 0.764028 rpy=-1.5708 2.36686e-13 -7.66952e-17
- joint arm_left_shoulder_roll_joint: limit lower=-1.5708 upper=-0 effort=20 velocity=15 -> lower=-0.261799 upper=1.309 effort=20 velocity=15; origin xyz=0.0255 0 0.043 rpy=1.5708 1.309 1.5708 -> xyz=0.0255 -1.44329e-15 0.043 rpy=1.5708 1.309 1.5708
- joint arm_left_shoulder_yaw_joint: origin xyz=0 0.123 -0.0255 rpy=-1.5708 0 0 -> xyz=2.77001e-14 0.123 -0.0255 rpy=-1.5708 5.43678e-13 5.82627e-14
- joint arm_right_elbow_pitch_joint: origin xyz=0.0245 0 0.043 rpy=1.5708 0 1.5708 -> xyz=0.0245 6.99949e-15 0.043 rpy=1.5708 1.198e-14 1.5708
- joint arm_right_elbow_roll_joint: origin xyz=0 0.123 -0.0255 rpy=1.5708 0 -3.14159 -> xyz=3.07195e-14 0.123 -0.0255 rpy=1.5708 3.84599e-15 -3.14159
- joint arm_right_shoulder_pitch_joint: origin xyz=0 -0.133 0.164028 rpy=-1.5708 0 -3.14159 -> xyz=1.14127e-16 -0.133 0.764028 rpy=-1.5708 -5.46706e-15 -3.14159
- joint arm_right_shoulder_roll_joint: limit lower=-0 upper=1.5708 effort=20 velocity=15 -> lower=-1.309 upper=0.261799 effort=20 velocity=15; origin xyz=-0.0255 0 0.043 rpy=1.5708 -1.309 -1.5708 -> xyz=-0.0255 3.21965e-15 0.043 rpy=1.5708 -1.309 -1.5708
- joint arm_right_shoulder_yaw_joint: origin xyz=0 0.123 -0.0255 rpy=1.5708 0 3.14159 -> xyz=8.10463e-15 0.123 -0.0255 rpy=1.5708 -1.73988e-13 3.14159
- joint imu: child imu -> imu_2; origin xyz=0.061722 0 0.08 rpy=0 0 0 -> xyz=0.061722 -1.49319e-16 0.68 rpy=-6.12323e-17 2.26485e-14 -2.65724e-15
- joint leg_left_ankle_pitch_joint: origin xyz=0 -0.16 -0.003 rpy=0 0 -3.14159 -> xyz=-2.44769e-15 -0.16 -0.003 rpy=1.34337e-14 -1.32117e-14 -3.14159
- joint leg_left_ankle_roll_joint: origin xyz=0.03 0.05 0.025 rpy=0 1.5708 0 -> xyz=0.03 0.05 0.025 rpy=-6.80837e-17 1.5708 0
- joint leg_left_hip_pitch_joint: origin xyz=0.027 0 0.052 rpy=1.5708 -0.785398 -1.5708 -> xyz=0.027 -1.11022e-16 0.052 rpy=1.5708 -0.785398 -1.5708
- joint leg_left_hip_roll_joint: origin xyz=-0.0290919 0.08 -0.057369 rpy=0 0.785398 0 -> xyz=-0.0290919 0.08 0.542631 rpy=2.21613e-15 0.785398 -7.34556e-15
- joint leg_left_hip_yaw_joint: origin xyz=0.027 0 -0.052 rpy=-1.5708 0 -1.5708 -> xyz=0.027 0 -0.052 rpy=-1.5708 -1.63347e-15 -1.5708
- joint leg_left_knee_pitch_joint: limit lower=0 upper=2.44346 effort=20 velocity=15 -> lower=-3.16192e-13 upper=2.44346 effort=20 velocity=15; origin xyz=0 0.15 -0.018 rpy=0 0 -3.14159 -> xyz=4.04191e-16 0.15 -0.018 rpy=1.40516e-29 1.72255e-16 -3.14159
- joint leg_right_ankle_pitch_joint: origin xyz=0 0.16 0.003 rpy=0 0 0 -> xyz=1.42421e-15 0.16 0.003 rpy=-2.22045e-16 -1.60812e-16 -1.12257e-13
- joint leg_right_ankle_roll_joint: origin xyz=0.03 0.05 -0.025 rpy=0 1.5708 0 -> xyz=0.03 0.05 -0.025 rpy=-6.80837e-17 1.5708 0
- joint leg_right_hip_pitch_joint: origin xyz=-0.027 0 0.052 rpy=1.5708 -0.785398 -1.5708 -> xyz=-0.027 -2.22045e-16 0.052 rpy=1.5708 -0.785398 -1.5708
- joint leg_right_hip_roll_joint: origin xyz=-0.0290919 -0.08 -0.057369 rpy=0 -0.785398 3.14159 -> xyz=-0.0290919 -0.08 0.542631 rpy=-1.75261e-15 -0.785398 3.14159
- joint leg_right_hip_yaw_joint: origin xyz=-0.027 0 -0.052 rpy=-1.5708 0 1.5708 -> xyz=-0.027 -1.38778e-17 -0.052 rpy=-1.5708 4.7846e-16 1.5708
- joint leg_right_knee_pitch_joint: limit lower=-0 upper=2.44346 effort=20 velocity=15 -> lower=-1.08358e-13 upper=2.44346 effort=20 velocity=15; origin xyz=0 0.15 0.018 rpy=0 0 0 -> xyz=0 0.15 0.018 rpy=3.21091e-16 2.40745e-16 8.46265e-17

File: data/urdf/berkeley_humanoid_lite_biped.urdf (robot description, URDF)
Before this commit: robot berkeley-humanoid-lite, 14 links, 13 joints
Links:
- added link imu_2, mass 0.00197704; visual mesh filename=./assets/merged/imu_2_visual.stl
- link base: mass 4.47154 -> 3.16059; geometry collision box size=0.15 0.14 0.23; visual mesh filename=./assets/merged/base_visual.stl
- link imu: mass 0.00197704 -> 1e-9; geometry 
- link leg_left_ankle_pitch: geometry visual mesh filename=./assets/merged/leg_left_ankle_pitch_visual.stl
- link leg_left_ankle_roll: mass 0.671532 -> 0.706476; geometry collision box size=0.072 0.22 0.04; visual mesh filename=./assets/merged/leg_left_ankle_roll_visual.stl
- link leg_left_hip_pitch: geometry collision cylinder length=0.13 radius=0.05; visual mesh filename=./assets/merged/leg_left_hip_pitch_visual.stl
- link leg_left_hip_roll: geometry visual mesh filename=./assets/merged/leg_left_hip_roll_visual.stl
- link leg_left_hip_yaw: geometry visual mesh filename=./assets/merged/leg_left_hip_yaw_visual.stl
- link leg_left_knee_pitch: geometry collision cylinder length=0.15 radius=0.04; visual mesh filename=./assets/merged/leg_left_knee_pitch_visual.stl
- link leg_right_ankle_pitch: geometry visual mesh filename=./assets/merged/leg_right_ankle_pitch_visual.stl
- link leg_right_ankle_roll: mass 0.671532 -> 0.706476; geometry collision box size=0.072 0.22 0.04; visual mesh filename=./assets/merged/leg_right_ankle_roll_visual.stl
- link leg_right_hip_pitch: geometry collision cylinder length=0.13 radius=0.05; visual mesh filename=./assets/merged/leg_right_hip_pitch_visual.stl
- link leg_right_hip_roll: geometry visual mesh filename=./assets/merged/leg_right_hip_roll_visual.stl
- link leg_right_hip_yaw: geometry visual mesh filename=./assets/merged/leg_right_hip_yaw_visual.stl
- link leg_right_knee_pitch: geometry collision cylinder length=0.15 radius=0.04; visual mesh filename=./assets/merged/leg_right_knee_pitch_visual.stl
Joints:
- added joint imu_frame: type fixed, parent imu_2, child imu, origin xyz=0 -6.33816e-19 0.005 rpy=0 -0 -1.90898e-31, axis 0 0 0
- joint imu: child imu -> imu_2; origin xyz=0.061722 0 0.08 rpy=0 0 0 -> xyz=0.061722 -1.49319e-16 0.68 rpy=-6.12323e-17 2.26485e-14 -2.65724e-15
- joint leg_left_ankle_pitch_joint: origin xyz=0 -0.16 -0.003 rpy=0 0 -3.14159 -> xyz=-2.44769e-15 -0.16 -0.003 rpy=1.34337e-14 -1.32117e-14 -3.14159
- joint leg_left_ankle_roll_joint: origin xyz=0.03 0.05 0.025 rpy=0 1.5708 0 -> xyz=0.03 0.05 0.025 rpy=-6.80837e-17 1.5708 0
- joint leg_left_hip_pitch_joint: origin xyz=0.027 0 0.052 rpy=1.5708 -0.785398 -1.5708 -> xyz=0.027 -1.11022e-16 0.052 rpy=1.5708 -0.785398 -1.5708
- joint leg_left_hip_roll_joint: origin xyz=-0.0290919 0.08 -0.057369 rpy=0 0.785398 0 -> xyz=-0.0290919 0.08 0.542631 rpy=2.21613e-15 0.785398 -7.34556e-15
- joint leg_left_hip_yaw_joint: origin xyz=0.027 0 -0.052 rpy=-1.5708 0 -1.5708 -> xyz=0.027 0 -0.052 rpy=-1.5708 -1.63347e-15 -1.5708
- joint leg_left_knee_pitch_joint: limit lower=0 upper=2.44346 effort=20 velocity=15 -> lower=-3.16192e-13 upper=2.44346 effort=20 velocity=15; origin xyz=0 0.15 -0.018 rpy=0 0 -3.14159 -> xyz=4.04191e-16 0.15 -0.018 rpy=1.40516e-29 1.72255e-16 -3.14159
- joint leg_right_ankle_pitch_joint: origin xyz=0 0.16 0.003 rpy=0 0 0 -> xyz=1.42421e-15 0.16 0.003 rpy=-2.22045e-16 -1.60812e-16 -1.12257e-13
- joint leg_right_ankle_roll_joint: origin xyz=0.03 0.05 -0.025 rpy=0 1.5708 0 -> xyz=0.03 0.05 -0.025 rpy=-6.80837e-17 1.5708 0
- joint leg_right_hip_pitch_joint: origin xyz=-0.027 0 0.052 rpy=1.5708 -0.785398 -1.5708 -> xyz=-0.027 -2.22045e-16 0.052 rpy=1.5708 -0.785398 -1.5708
- joint leg_right_hip_roll_joint: origin xyz=-0.0290919 -0.08 -0.057369 rpy=0 -0.785398 3.14159 -> xyz=-0.0290919 -0.08 0.542631 rpy=-1.75261e-15 -0.785398 3.14159
- joint leg_right_hip_yaw_joint: origin xyz=-0.027 0 -0.052 rpy=-1.5708 0 1.5708 -> xyz=-0.027 -1.38778e-17 -0.052 rpy=-1.5708 4.7846e-16 1.5708
- joint leg_right_knee_pitch_joint: limit lower=-0 upper=2.44346 effort=20 velocity=15 -> lower=-1.08358e-13 upper=2.44346 effort=20 velocity=15; origin xyz=0 0.15 0.018 rpy=0 0 0 -> xyz=0 0.15 0.018 rpy=3.21091e-16 2.40745e-16 8.46265e-17

Commit message: UPDATE: larger joint range for teleop

File: data/urdf/berkeley_humanoid_lite.urdf (robot description, URDF)
Before this commit: robot berkeley-humanoid-lite, 27 links, 26 joints
Joints:
- joint arm_left_elbow_roll_joint: limit lower=-0.785398 upper=0.785398 effort=20 velocity=15 -> lower=-1.5708 upper=1.5708 effort=20 velocity=15
- joint arm_left_shoulder_pitch_joint: limit lower=-1.5708 upper=0.785398 effort=20 velocity=15 -> lower=-2.35619 upper=1.5708 effort=20 velocity=15
- joint arm_left_shoulder_yaw_joint: limit lower=-0.785398 upper=0.785398 effort=20 velocity=15 -> lower=-1.5708 upper=1.5708 effort=20 velocity=15
- joint arm_right_elbow_roll_joint: limit lower=-0.785398 upper=0.785398 effort=20 velocity=15 -> lower=-1.5708 upper=1.5708 effort=20 velocity=15
- joint arm_right_shoulder_pitch_joint: limit lower=-0.785398 upper=1.5708 effort=20 velocity=15 -> lower=-1.5708 upper=2.35619 effort=20 velocity=15
- joint arm_right_shoulder_yaw_joint: limit lower=-0.785398 upper=0.785398 effort=20 velocity=15 -> lower=-1.5708 upper=1.5708 effort=20 velocity=15
